File: firststep1/driver.kicad_sch (KiCad schematic)
At the start: 3 parts, among them M1 Motor_DC, Q1 IRF540N

Commit message: minor
Parts:
- gave numbers to parts that had none: 1
Changed lines of the file:
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@@
   (symbol (lib_id "Relay:G5LE-1") (at 75.946 105.41 0) (unit 1)
     (in_bom yes) (on_board yes) (fields_autoplaced)
-    (property "Reference" "K?" (id 0) (at 87.63 104.1399 0)
+    (property "Reference" "K1" (id 0) (at 87.63 104.1399 0)
       (effects (font (size 1.27 1.27)) (justify left))
     )
